Commit message: Se añadio a la visualizacion en Rviz el soporte de la camapra

File: phantom_ws/src/phantomx_pincher_description/urdf/kit.xacro (robot description, xacro)
@@ -242,4 +242,22 @@
     <child link="canecaFrontalIzquierda_link" />
     <origin xyz="0.19397558339 0.09252160722 0.016" rpy="0 0 0" />
+  </joint>
+  <!-- ============================= -->
+  <!-- 📷 Soporte de Cámara -->
+  <!-- ============================= -->
+  <link name="soporteCamara_link">
+    <visual>
+      <origin xyz="0 0 0" rpy="0 0 -${PI/2}" />
+      <geometry>
+        <mesh filename="package://phantomx_pincher_description/meshes/STL/ensambleSoporteCamara.stl"
+              scale="0.001 0.001 0.001" />
+      </geometry>
+      <material name="gray" />
+    </visual>
+  </link>
+  <joint name="base_soporteCamara_joint" type="fixed">
+    <parent link="baseFija_link" />
+    <child link="soporteCamara_link" />
+    <origin xyz="0.26 0.0 0.009" rpy="0 0 0" />
   </joint>
   <!-- ============================= -->
