Commit message: Calibracion motores, puerto configurable, API bajo demanda y credenciales via .env

File: phantom_ws/src/phantomx_pincher_description/urdf/phantomx_pincher.urdf (robot description, URDF)
Before this commit: robot phantomx_pincher, 35 links, 34 joints
Links:
- added link soporteCamara_link; visual mesh filename=package://phantomx_pincher_description/meshes/STL/ensambleS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 scale=0.001 0.001 0.001
Joints:
- added joint base_soporteCamara_joint: type fixed, parent baseFija_link, child soporteCamara_link, origin xyz=0.26 0.0 0.009 rpy=0 0 0
